Commit message: package ready

File: urdf/erl1.urdf (robot description, URDF)
Before this commit: robot erl1, 3 links, 2 joints
Links:
- link link_chassis: geometry collision box size=0.5 0.3 0.07; collision sphere radius=0.05

Commit message: update after class

File: urdf/erl1.urdf (robot description, URDF)
Before this commit: robot erl1, 3 links, 2 joints
Links:
- link link_chassis: geometry collision mesh filename=package://erl1/meshes/mogi_bot.dae; collision sphere radius=0.05
