Commit message: package updated 2026-2027

File: urdf/my_robot.urdf (robot description, URDF)
Before this commit: robot erl1, 4 links, 3 joints
Links:
- removed link link_cube
- added link camera_link, mass 0.3; collision box size=0.1 0.1 0.1; visual box size=0.1 0.1 0.1
- added link camera_link_optical
- added link imu_link
Joints:
- removed joint cube_joint
- added joint camera_joint: type revolute, parent link_chassis, child camera_link, origin xyz=0 0 0.035 rpy=0 0 0, axis 0 0 1, limit lower=-1.57 upper=1.57 effort=5 velocity=1.0
- added joint camera_optical_joint: type fixed, parent camera_link, child camera_link_optical, origin xyz=0 0 0 rpy=-1.5707 0 -1.5707
- added joint imu_joint: type fixed, parent link_chassis, child imu_link, origin xyz=0 0 0 rpy=0 0 0

Commit message: assignment added

File: urdf/my_robot.urdf (robot description, URDF)
Before this commit: robot erl1, 6 links, 5 joints
Links:
- added link scan_link, mass 1e-5; collision box size=.1 .1 .1; visual cylinder length=0.1 radius=0.05
Joints:
- added joint scan_joint: type fixed, parent link_chassis, child scan_link, origin xyz=-0.2 0 0.19 rpy=0 0 0
- joint camera_joint: origin xyz=0 0 0.035 rpy=0 0 0 -> xyz=0.3 0 0.035 rpy=0 0 0
